File: Backplane PCB/1U Backplane.kicad_pcb (KiCad board)
At the start: 4 copper layers, 165 x 43.5 mm, 34 parts, among them J1 SATA 7+15 Female, J2 SATA 7+15 Male, J3 Molex 470533000, J4 SATA 7+15 Female, J5 SATA 7+15 Male, J6 Molex 470533000, Q1 BSS138, U1 SN74LV1T34DBV, U2 SN74LV1T34DBV, U3 MIC1557YM5

Commit message: Update PCB
Parts:
- added R3: 0, Resistor_SMD:R_0402_1005Metric, B.Cu at (172.9, 115.9)
- added R7: 0, Resistor_SMD:R_0402_1005Metric, B.Cu at (157.9, 97.0)
- D4: value 2.8V -> 2.8V / 10mA
- D5: renamed from D6; value 2.0V -> BZX38450-C1V8X
- D6: renamed from D5; value 2.8V -> 2.8V / 10mA
- D7: renamed from D1; value 2.8V -> 2.8V / 10mA
- D8: renamed from D3; value 2.0V -> BZX38450-C1V8X
- D9: renamed from D2; value 2.8V -> 2.8V / 10mA
- R1: renamed from R4; value 150 -> 220
- R2: renamed from R5; value 16.9k -> 17.8k
- R4: renamed from R6; value 150 -> 220
- R5: renamed from R1; value 150 -> 220
- R6: renamed from R2; value 16.9k -> 17.8k
- R8: renamed from R3; value 150 -> 220
- renumbered C3 to C1, C4 to C2, C2 to C3, C1 to C4, D8 to D1, D7 to D2, D9 to D3, J4 to J1, J5 to J2, J6 to J3, J1 to J4, J2 to J5, J3 to J6, U3 to U1, U1 to U3
Connections:
- D5 pad 1: /Left Drive/RESERVED -> /Left Drive/RESERVED_DRIVE
- D8 pad 1: /Right Drive/RESERVED -> /Right Drive/RESERVED_DRIVE
- J1 pad 18: /Left Drive/RESERVED -> /Left Drive/RESERVED_DRIVE
- J2 pad 18: /Left Drive/RESERVED -> /Left Drive/RESERVED_HOST
- J4 pad 18: /Right Drive/RESERVED -> /Right Drive/RESERVED_DRIVE
- J5 pad 18: /Right Drive/RESERVED -> /Right Drive/RESERVED_HOST
- R2 pad 2: /Left Drive/RESERVED -> /Left Drive/RESERVED_DRIVE
- R6 pad 2: /Right Drive/RESERVED -> /Right Drive/RESERVED_DRIVE
- U2 pad 2: /Left Drive/RESERVED -> /Left Drive/RESERVED_DRIVE
- U3 pad 2: /Right Drive/RESERVED -> /Right Drive/RESERVED_DRIVE
Routing:
- net /Right Drive/RESERVED: track 107.5 -> 0.00 mm
- net /Right Drive/RESERVED_DRIVE: track 0.00 -> 105.7 mm
- net /Left Drive/RESERVED: track 32.6 -> 0.00 mm
- net /Left Drive/RESERVED_DRIVE: track 0.00 -> 29.6 mm
- net /Left Drive/RESERVED_HOST: track 0.00 -> 2.29 mm
- net /Right Drive/RESERVED_HOST: track 0.00 -> 1.36 mm
