File: Backplane PCB/1U Backplane.kicad_sch (KiCad schematic)
At the start: 8 parts, among them Q1 BSS138, U3 MIC1557YM5

Commit message: Update PCB
Parts:
- renumbered C3 to C1, C4 to C2, D8 to D1, D7 to D2, D9 to D3, U3 to U1
Other:
- moved on the sheet: C1, C2, D1, D2, D3, Q1, RV1, U1
