File: Backplane PCB/Drive.kicad_sch (KiCad schematic)
At the start: 11 parts, among them J4 SATA 7+15 Female, J5 SATA 7+15 Male, J6 Molex 470533000, U2 SN74LV1T34DBV

Commit message: Update PCB
Parts:
- removed C2: 100n, Capacitor_SMD:C_0603_1608Metric_Pad1.08x0.95mm_HandSolder, symbol Device:C_Small
- removed D5: 2.8V, LED_SMD:LED_0603_1608Metric_Pad1.05x0.95mm_HandSolder, symbol Device:LED
- removed D6: 2.0V, Diode_SMD:D_SOD-323_HandSoldering, symbol Device:D_Zener
- removed R6: 150, Resistor_SMD:R_0603_1608Metric_Pad0.98x0.95mm_HandSolder, symbol Device:R_US
- added C3: 100n, Capacitor_SMD:C_0603_1608Metric_Pad1.08x0.95mm_HandSolder, symbol Device:C_Small
- added D5: BZX38450-C1V8X, Diode_SMD:D_SOD-323_HandSoldering, symbol Device:D_Zener
- added D6: 2.8V / 10mA, LED_SMD:LED_0603_1608Metric_Pad1.05x0.95mm_HandSolder, symbol Device:LED
- added R3: 0, Resistor_SMD:R_0402_1005Metric, symbol Device:R_US
- added R4: 220, Resistor_SMD:R_0603_1608Metric_Pad0.98x0.95mm_HandSolder, symbol Device:R_US
- D4: value 2.8V -> 2.8V / 10mA
- R1: renamed from R4; value 150 -> 220
- R2: renamed from R5; value 16.9k -> 17.8k
- renumbered J4 to J1, J5 to J2, J6 to J3
Connections:
- net +5V: now also C3.1, D6.2 (A)
- net GNDPWR: now also C3.2, D5.2 (A)
- net at U2.4 (Y): now also R4.2
- net RESERVED renamed RESERVED_DRIVE
- net RESERVED_DRIVE: now also D5.1 (K), R3.1; no longer J2.18
- new net: D6.1 (K), R4.1
- new net RESERVED_HOST: J2.18, R3.2
Other:
- note added: "Note: R3 is DNI because many SATA cables, extensions, etc, just ground the RESERVED pin, which prevents the drive's activity signal from toggling. Leaving it open allows the drive to toggle the activity LED, but will prevent staggered spinup from being enabled (where drive media is not spun up on powerup but insteads waits for data transmission). If staggered spinup is required, populate R3, keep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"
- note added: "Note: this driver circuit is one of the suggestions in the SATA spec The max high voltage on RESERVED_DRIVE is 2.1V, but the minimum input high voltage for the level shifter is ~2V (at 5V Vcc). It's hard to meet this perfectly across all extremes of the zener voltage, supply, and temp. The zener is spec'd at 1.8V nominal at 50uA. It is biased closer to 300uA for fastest edge rates and also to kee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"
- moved on the sheet: J1, J2, U2
